Commit message: Add files via upload
modified urdf

File: bot.urdf (robot description, URDF)
Before this commit: robot bot, 8 links, 7 joints
Joints:
- removed joint armbase_link1
- removed joint basebase
- removed joint link12
- added joint armbase_to_link1: type continuous, parent armbase, child armlink1, origin xyz=0 0 0.05 rpy=0 0 0, axis 0 0 1
- added joint base_to_armbase: type fixed, parent base_link, child armbase, origin xyz=0 0 0.05 rpy=0 0 0
- added joint link1_to_link2: type revolute, parent armlink1, child armlink2, origin xyz=0 0 0.5 rpy=0 0 0, axis 0 1 0, limit lower=-1.57 upper=1.57 effort=10 velocity=1.0
